Commit message: Preserve concave robot clearances in native simulation models
Decompose every concave manufacturer collision mesh through the existing offline CoACD build. Cover each physical link once for conservative planning bounds, independent of native convex partitions. Preserve the visual meshes, inertias, joints and collision exclusions.

Validate folded YAM forearm clearance, whole-triangle coverage and partition invariance. SDK: 516 passed, 7 skipped; MuJoCo jog panels: 2 passed; normal MuJoCo/SAPIEN tools and authored programs: 4 passed. SAPIEN jog timing remains under investigation; Isaac native execution awaits operator license acceptance.

Co-Authored-By: Claude Fable 5 <noreply@anthropic.com>

File: sdk/python/waddle_sdk/simulators/data/xarm7/robot.urdf (robot description, URDF)
Before this commit: robot xarm7_g2, 16 links, 15 joints
Links:
- link left_inner_knuckle: geometry collision mesh filename=assets/collision/left_inner_knuckle/left_inner_knuckle-0.stl; collision mesh filename=assets/collision/left_inner_knuckle/left_inner_knuckle-1.stl
- link left_outer_knuckle: geometry collision mesh filename=assets/collision/left_outer_knuckle/left_outer_knuckle-0.stl; collision mesh filename=assets/collision/left_outer_knuckle/left_outer_knuckle-1.stl
- link link1: geometry collision mesh filename=assets/collision/link1/link1-0.stl; collision mesh filename=assets/collision/link1/link1-1.stl
- link link2: geometry collision mesh filename=assets/collision/link2/link2-0.stl; collision mesh filename=assets/collision/link2/link2-1.stl
- link link3: geometry collision mesh filename=assets/collision/link3/link3-0.stl; collision mesh filename=assets/collision/link3/link3-1.stl
- link link4: geometry collision mesh filename=assets/collision/link4/link4-0.stl; collision mesh filename=assets/collision/link4/link4-1.stl
- link link5: geometry collision mesh filename=assets/collision/link5/link5-0.stl; collision mesh filename=assets/collision/link5/link5-1.stl
- link link6: geometry collision mesh filename=assets/collision/link6/link6-0.stl; collision mesh filename=assets/collision/link6/link6-1.stl
- link link7: geometry collision mesh filename=assets/collision/link7/link7-0.stl; collision mesh filename=assets/collision/link7/link7-1.stl
- link link_base: geometry collision mesh filename=assets/collision/link_base/link_base-0.stl; collision mesh filename=assets/collision/link_base/link_base-1.stl
- link right_inner_knuckle: geometry collision mesh filename=assets/collision/right_inner_knuckle/right_inner_knuckle-0.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; collision mesh filename=assets/collision/right_inner_knuckle/right_inner_knuckle-1.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
- link right_outer_knuckle: geometry collision mesh filename=assets/collision/right_outer_knuckle/right_outer_knuckle-0.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; collision mesh filename=assets/collision/right_outer_knuckle/right_outer_knuckle-1.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

File: sdk/python/waddle_sdk/simulators/data/yam/robot.urdf (robot description, URDF)
Before this commit: robot yam_v0, 11 links, 10 joints
Links:
- link base_link: geometry collision mesh filename=assets/collision/base_link/base_link-0.stl; collision mesh filename=assets/collision/base_link/base_link-1.stl
- link gripper: geometry collision mesh filename=assets/collision/gripper/gripper-0.stl; collision mesh filename=assets/collision/gripper/gripper-1.stl
- link link_1: geometry collision mesh filename=assets/collision/link_1/link_1-0.stl; collision mesh filename=assets/collision/link_1/link_1-1.stl
- link link_2: geometry collision mesh filename=assets/collision/link_2/link_2-0.stl; collision mesh filename=assets/collision/link_2/link_2-1.stl
- link link_3: geometry collision mesh filename=assets/collision/link_3/link_3-0.stl; collision mesh filename=assets/collision/link_3/link_3-1.stl
- link link_4: geometry collision mesh filename=assets/collision/link_4/link_4-0.stl; collision mesh filename=assets/collision/link_4/link_4-1.stl
- link link_5: geometry collision mesh filename=assets/collision/link_5/link_5-0.stl; collision mesh filename=assets/collision/link_5/link_5-1.stl
